Commit message: clean the test file

File: robots/kuka_iiwa_14/iiwa14.urdf (robot description, URDF)
Before this commit: robot iiwa14, 10 links, 9 joints
Links:
- link iiwa_link_0: geometry collision mesh filename=meshes/iiwa14/collision/link_0.stl; visual mesh filename=meshes/iiwa14/visual/link_0.stl
- link iiwa_link_1: geometry collision mesh filename=meshes/iiwa14/collision/link_1.stl; visual mesh filename=meshes/iiwa14/visual/link_1.stl
- link iiwa_link_2: geometry collision mesh filename=meshes/iiwa14/collision/link_2.stl; visual mesh filename=meshes/iiwa14/visual/link_2.stl
- link iiwa_link_3: geometry collision mesh filename=meshes/iiwa14/collision/link_3.stl; visual mesh filename=meshes/iiwa14/visual/link_3.stl
- link iiwa_link_4: geometry collision mesh filename=meshes/iiwa14/collision/link_4.stl; visual mesh filename=meshes/iiwa14/visual/link_4.stl
- link iiwa_link_5: geometry collision mesh filename=meshes/iiwa14/collision/link_5.stl; visual mesh filename=meshes/iiwa14/visual/link_5.stl
- link iiwa_link_6: geometry collision mesh filename=meshes/iiwa14/collision/link_6.stl; visual mesh filename=meshes/iiwa14/visual/link_6.stl
- link iiwa_link_7: geometry collision mesh filename=meshes/iiwa14/collision/link_7.stl; visual mesh filename=meshes/iiwa14/visual/link_7.stl
