Commit message: Uncomment collision tags

File: robots/kuka_lwr_force/kuka.urdf (robot description, URDF)
Before this commit: robot kuka, 12 links, 11 joints
Links:
- link adaptor_kuka: geometry collision mesh filename=meshes/visual/adaptor_kuka.stl scale=0.001 0.001 0.001; visual mesh filename=meshes/visual/adaptor_kuka.stl scale=0.001 0.001 0.001
- link force_torque_sensor: geometry collision cylinder length=0.0333 radius=0.04; visual mesh filename=meshes/visual/force_sensor.stl scale=0.001 0.001 0.001
- link lwr_arm_0_link: geometry collision cylinder length=0.11 radius=0.07; visual mesh filename=meshes/visual/base.STL
- link lwr_arm_1_link: geometry collision cylinder length=0.208 radius=0.07; collision sphere radius=0.07
- link lwr_arm_2_link: geometry collision cylinder length=0.208 radius=0.07; collision sphere radius=0.07
- link lwr_arm_3_link: geometry collision cylinder length=0.208 radius=0.07; collision sphere radius=0.07
- link lwr_arm_4_link: geometry collision cylinder length=0.208 radius=0.07; collision sphere radius=0.07
- link lwr_arm_5_link: geometry collision cylinder length=0.198 radius=0.07; collision sphere radius=0.07
- link lwr_arm_7_link: geometry collision cylinder length=0.046 radius=0.04; visual cylinder length=0.03 radius=0.033

Commit message: Intermediate commit regarding interpolation node, working but with non-generalised code patches

File: robots/kuka_lwr_force/kuka.urdf (robot description, URDF)
Before this commit: robot kuka, 12 links, 11 joints
Links:
- added link end_effector_ball; visual sphere radius=0.015
- link end_effector_sponge: geometry collision cylinder length=0.25 radius=0.005; visual cylinder length=0.25 radius=0.005
Joints:
- added joint end_effector_ball: type fixed, parent end_effector_sponge, child end_effector_ball, origin xyz=0 0 0.12 rpy=0 0 0.0

Commit message: Reverting edits on Kuka URDF file (mistake)

File: robots/kuka_lwr_force/kuka.urdf (robot description, URDF)
Before this commit: robot kuka, 13 links, 12 joints
Links:
- removed link end_effector_ball
- link end_effector_sponge: geometry collision cylinder length=0.015 radius=0.04; visual cylinder length=0.015 radius=0.04
Joints:
- removed joint end_effector_ball

Commit message: Added world link for the LWR, cause it position w.r.t the world had offset

File: robots/kuka_lwr_force/kuka.urdf (robot description, URDF)
Before this commit: robot kuka, 12 links, 11 joints
Links:
- added link lwr_world, mass 0
Joints:
- added joint lwr_world_joint: type fixed, parent lwr_world, child lwr_arm_0_link, origin xyz=0 0 0 rpy=0 0 0
