Commit message: Updates in the configs yaml launch files for real robot/vicon exp

File: robots/kuka_lwr_force/kuka_push_visual.urdf (robot description, URDF)
Before this commit: robot kuka, 13 links, 12 joints
Links:
- link adaptor_kuka: geometry visual mesh filename=meshes/visual/adaptor_kuka.stl scale=0.001 0.001 0.001
- link end_effector_ball: geometry visual sphere radius=0.013
- link force_torque_sensor: geometry visual mesh filename=meshes/visual/force_sensor.stl scale=0.001 0.001 0.001
- link lwr_arm_0_link: geometry visual mesh filename=meshes/visual/base.STL
- link lwr_arm_1_link: geometry visual mesh filename=meshes/visual/link_1.STL
- link lwr_arm_2_link: geometry visual mesh filename=meshes/visual/link_2.STL
- link lwr_arm_3_link: geometry visual mesh filename=meshes/visual/link_3.STL
- link lwr_arm_4_link: geometry visual mesh filename=meshes/visual/link_4.STL
- link lwr_arm_5_link: geometry visual mesh filename=meshes/visual/link_5.STL
- link lwr_arm_7_link: geometry visual cylinder length=0.03 radius=0.033; visual mesh filename=meshes/visual/link_7.STL
