Commit message: Tunning parameters for pushing example

File: robots/kuka_lwr_force/kuka_push.urdf (robot description, URDF)
Before this commit: robot kuka, 13 links, 12 joints
Links:
- link end_effector_ball: mass None -> 0.05; geometry collision sphere radius=0.015; visual sphere radius=0.015
- link end_effector_sponge: geometry visual cylinder length=0.25 radius=0.005

Commit message: Change tool sphere radious

File: robots/kuka_lwr_force/kuka_push.urdf (robot description, URDF)
Before this commit: robot kuka, 13 links, 12 joints
Links:
- link end_effector_ball: geometry collision sphere radius=0.013; visual sphere radius=0.013

File: robots/kuka_lwr_force/kuka_push_visual.urdf (robot description, URDF)
Before this commit: robot kuka, 13 links, 12 joints
Links:
- link end_effector_ball: geometry visual sphere radius=0.016
