Commit message: Update on parameter files

File: robots/cloth/cloth.urdf (robot description, URDF)
Before this commit: robot cloth, 4 links, 3 joints
Joints:
- joint Cyl1_Cyl2: limit lower=-2.0001 upper=2.0001 effort=10 velocity=1.0 -> lower=-0.2001 upper=0.2001 effort=100 velocity=1.0
- joint Cyl1_Cyl3: limit lower=-2.0001 upper=2.0001 effort=10 velocity=1.0 -> lower=-0.2001 upper=0.2001 effort=100 velocity=1.0
- joint Cyl3_Cyl4: axis (none) -> 0 1 0; limit (none) -> lower=-0.25 upper=0.0 effort=75 velocity=1.0; type fixed -> prismatic

File: robots/human_model/humanSubject02_48dof.urdf (robot description, URDF)
Before this commit: robot XSensStyleModel_template, 49 links, 48 joints
Links:
- link Head: mass 2.8584 -> 0.8584
- link RightForeArm_f1: geometry collision sphere radius=0.023
- link RightUpperArm: geometry collision cylinder length=0.27379 radius=0.02014; visual cylinder length=0.27379 radius=0.0300014
Joints:
- joint jC1Head_rotx: limit lower=-0.610865 upper=0.610865 effort=30 velocity=1.0 -> lower=-0.610865 upper=0.610865 effort=500 velocity=1.0
- joint jC1Head_roty: limit lower=-0.436332 upper=0.174533 effort=30 velocity=1.0 -> lower=-0.436332 upper=0.174533 effort=500 velocity=1.0
- joint jL1T12_rotx: limit lower=-0.610865 upper=0.610865 effort=30 velocity=1.0 -> lower=-0.610865 upper=0.610865 effort=500 velocity=1.0
- joint jL1T12_roty: limit lower=-0.523599 upper=1.309 effort=30 velocity=1.0 -> lower=-0.523599 upper=1.309 effort=500 velocity=1.0
- joint jL4L3_rotx: limit lower=-0.610865 upper=0.610865 effort=30 velocity=1.0 -> lower=-0.610865 upper=0.610865 effort=500 velocity=1.0
- joint jL4L3_roty: limit lower=-0.523599 upper=1.309 effort=30 velocity=1.0 -> lower=-0.523599 upper=1.309 effort=500 velocity=1.0
- joint jL5S1_rotx: limit lower=-0.610865 upper=0.610865 effort=30 velocity=1.0 -> lower=-0.610865 upper=0.610865 effort=500 velocity=1.0
- joint jL5S1_roty: limit lower=-0.523599 upper=1.309 effort=30 velocity=1.0 -> lower=-0.523599 upper=1.309 effort=500 velocity=1.0
- joint jT1C7_roty: limit lower=-0.959931 upper=1.5708 effort=30 velocity=1.0 -> lower=-0.959931 upper=1.5708 effort=500 velocity=1.0
- joint jT1C7_rotz: limit lower=-1.22173 upper=1.22173 effort=30 velocity=1.0 -> lower=-1.22173 upper=1.22173 effort=500 velocity=1.0
- joint jT9T8_rotx: limit lower=-0.349066 upper=0.349066 effort=30 velocity=1.0 -> lower=-0.349066 upper=0.349066 effort=500 velocity=1.0
- joint jT9T8_roty: limit lower=-0.261799 upper=0.698132 effort=30 velocity=1.0 -> lower=-0.261799 upper=0.698132 effort=500 velocity=1.0
- joint jT9T8_rotz: limit lower=-0.610865 upper=0.610865 effort=30 velocity=1.0 -> lower=-0.610865 upper=0.610865 effort=500 velocity=1.0
