Commit message: Update of config, launch and URDF files

File: robots/human_model/humanSubject02_48dof.urdf (robot description, URDF)
Before this commit: robot XSensStyleModel_template, 49 links, 48 joints
Links:
- link RightUpperArm: geometry collision cylinder length=0.27379 radius=0.025014; visual cylinder length=0.27379 radius=0.0300014
Joints:
- joint jRightShoulder_rotx: limit lower=-2.35619 upper=1.5708 effort=30 velocity=1.0 -> lower=-2.35619 upper=1.5708 effort=30 velocity=0.2
- joint jRightShoulder_roty: limit lower=-1.5708 upper=1.5708 effort=30 velocity=1.0 -> lower=-1.5708 upper=1.5708 effort=30 velocity=0.2

Commit message: update configuration files after RAL submission

File: robots/human_model/humanSubject02_48dof.urdf (robot description, URDF)
Before this commit: robot XSensStyleModel_template, 49 links, 48 joints
Links:
- link Head: geometry collision sphere radius=0.09223; visual sphere radius=0.09223
- link LeftHand: geometry collision box size=0.11468 0.11202 0.040019; visual box size=0.11468 0.11202 0.040019
- link RightHand: geometry collision box size=0.11468 0.11202 0.040019; visual box size=0.11468 0.11202 0.040019
Joints:
- joint jLeftWrist_rotx: origin xyz=0.000133     0.22718           0 rpy=0 0 0 -> xyz=0.000133     0.19718           0 rpy=0 0 0
- joint jRightWrist_rotx: origin xyz=0.000133    -0.22718           0 rpy=0 0 0 -> xyz=0.000133    -0.19718           0 rpy=0 0 0
