Commit message: Update iiwa urdf and yin - yang yaml files to be used for the basic example and the IK example

File: robots/kuka_iiwa/iiwa14.urdf (robot description, URDF)
Before this commit: robot iiwa14, 10 links, 9 joints
Links:
- removed link iiwa_link_ee
- removed link world
- added link adaptor_kuka, mass 0.1; collision mesh filename=meshes/iiwa14/visual/adaptor_kuka.stl scale=0.001 0.001 0.001; visual mesh filename=meshes/iiwa14/visual/adaptor_kuka.stl scale=0.001 0.001 0.001
- added link end_effector, mass 1; collision mesh filename=meshes/iiwa14/visual/adaptor_endeffector.stl scale=0.001 0.001 0.001; visual mesh filename=meshes/iiwa14/visual/adaptor_endeffector.stl scale=0.001 0.001 0.001
- added link end_effector_sponge, mass 1; collision cylinder length=0.015 radius=0.04; visual cylinder length=0.015 radius=0.04
- added link force_torque_sensor, mass 0.5; collision cylinder length=0.0333 radius=0.04; visual mesh filename=meshes/iiwa14/visual/force_sensor.stl scale=0.001 0.001 0.001
- added link iiwa_world, mass 0
Joints:
- removed joint iiwa_joint_ee
- added joint end_effector_joint: type fixed, parent force_torque_sensor, child end_effector, origin xyz=0 0 0.02 rpy=0 0 0.0
- added joint end_effector_joint_sponge: type fixed, parent end_effector, child end_effector_sponge, origin xyz=0 0 0.015 rpy=0 0 0.0
- added joint force_torque_sensor_mount: type fixed, parent adaptor_kuka, child force_torque_sensor, origin xyz=0 0 0.0453 rpy=0 0 0
- added joint iiwa_joint_8: type fixed, parent iiwa_link_7, child adaptor_kuka, origin xyz=0 0 0.032 rpy=0 0 3.14159265359
- joint world_iiwa_joint: parent world -> iiwa_world

Commit message: IIWA urdf update, still is not correct

File: robots/kuka_iiwa/iiwa14.urdf (robot description, URDF)
Before this commit: robot iiwa14, 13 links, 12 joints
Links:
- link end_effector_sponge: geometry collision cylinder length=0.00001 radius=0.04; visual cylinder length=0.00001 radius=0.04

Commit message: Add hinge plate rotation to iiwa urdf

File: robots/kuka_iiwa/iiwa14.urdf (robot description, URDF)
Before this commit: robot iiwa14, 13 links, 12 joints
Links:
- added link iiwa_link_0_hinge, mass 0
- added link iiwa_world_hinge, mass 0
- link iiwa_link_0: geometry collision mesh filename=meshes/iiwa14/collision/link_0.stl; visual mesh filename=meshes/iiwa14/visual/link_0.stl
- link iiwa_world: geometry visual mesh filename=meshes/iiwa14/visual/base-Model.stl scale=0.001 0.001 0.001
Joints:
- removed joint world_iiwa_joint
- added joint base_hinge_joint: type fixed, parent iiwa_world_hinge, child iiwa_link_0_hinge, origin xyz=0 0 0 rpy=0 0.0 0
- added joint iiwa_link_0_hinge: type fixed, parent iiwa_link_0_hinge, child iiwa_link_0, origin xyz=-0.095 0 0.010 rpy=0 0 0
- added joint world_hinge_joint: type fixed, parent iiwa_world, child iiwa_world_hinge, origin xyz=0.090 0 0.045 rpy=0 0 0

Commit message: add base to the original urdf fils

File: robots/kuka_iiwa/iiwa14.urdf (robot description, URDF)
Before this commit: robot iiwa14, 15 links, 14 joints
Joints:
- joint base_hinge_joint: origin xyz=0 0 0 rpy=0 0.0 0 -> xyz=0 0 0 rpy=0 1.0472 0

File: robots/kuka_iiwa/iiwa14_visual.urdf (robot description, URDF)
Before this commit: robot iiwa14, 13 links, 12 joints
Links:
- added link iiwa_link_0_hinge, mass 0
- added link iiwa_world_hinge, mass 0
Joints:
- removed joint world_iiwa_joint
- added joint base_hinge_joint: type fixed, parent iiwa_world_hinge, child iiwa_link_0_hinge, origin xyz=0 0 0 rpy=0 1.0472 0
- added joint iiwa_link_0_hinge: type fixed, parent iiwa_link_0_hinge, child iiwa_link_0, origin xyz=-0.095 0 0.010 rpy=0 0 0
- added joint world_hinge_joint: type fixed, parent iiwa_world, child iiwa_world_hinge, origin xyz=0.090 0 0.045 rpy=0 0 0

Commit message: Update end-effector of the urdf

File: robots/kuka_iiwa/iiwa14.urdf (robot description, URDF)
Before this commit: robot iiwa14, 15 links, 14 joints
Links:
- removed link adaptor_kuka
- removed link end_effector
- added link adapter, mass 1; visual mesh filename=meshes/iiwa14/visual/schunk_adapter-Assembly.stl scale=0.001 0.001 0.001
- added link iiwa_link_ee, mass 0.000001
- link end_effector_sponge: geometry collision mesh filename=meshes/iiwa14/visual/adaptor_endeffector-Body.stl scale=0.001 0.001 0.001; visual mesh filename=meshes/iiwa14/visual/adaptor_endeffector-Body.stl scale=0.001 0.001 0.001
- link force_torque_sensor: geometry visual mesh filename=meshes/iiwa14/visual/ATI-Delta.stl scale=0.001 0.001 0.001
Joints:
- removed joint force_torque_sensor_mount
- removed joint iiwa_joint_8
- added joint iiwa_joint_ee: type fixed, parent iiwa_link_7, child iiwa_link_ee, origin xyz=0 0 0.045 rpy=0 0 0
- added joint iiwa_joint_ft: type fixed, parent iiwa_link_ee, child force_torque_sensor, origin xyz=0 0 0 rpy=0 0 1.57
- joint end_effector_joint: child end_effector -> adapter; origin xyz=0 0 0.02 rpy=0 0 0.0 -> xyz=0 0 0.033 rpy=0 0 0.0
- joint end_effector_joint_sponge: origin xyz=0 0 0.015 rpy=0 0 0.0 -> xyz=0 0 0.058 rpy=0 0 0.0; parent end_effector -> adapter

Commit message: Fix large stl files

File: robots/kuka_iiwa/iiwa14.urdf (robot description, URDF)
Before this commit: robot iiwa14, 15 links, 14 joints
Links:
- link adapter: geometry visual mesh filename=meshes/iiwa14/visual/schunk_adapter-Assembly_simplified.stl scale=0.001 0.001 0.001
- link end_effector_sponge: geometry collision mesh filename=meshes/iiwa14/visual/adaptor_endeffector-Body_simplified.stl scale=0.001 0.001 0.001; visual mesh filename=meshes/iiwa14/visual/adaptor_endeffector-Body_simplified.stl scale=0.001 0.001 0.001
- link force_torque_sensor: geometry visual mesh filename=meshes/iiwa14/visual/ATI-Delta_simplified.stl scale=0.001 0.001 0.001

Commit message: Custom change in URDF for safety check of the motion

File: robots/kuka_iiwa/iiwa14.urdf (robot description, URDF)
Before this commit: robot iiwa14, 15 links, 14 joints
Joints:
- joint end_effector_joint_sponge: origin xyz=0 0 0.058 rpy=0 0 0.0 -> xyz=0 0 0.078 rpy=0 0 0.0

File: robots/kuka_iiwa/iiwa14_visual.urdf (robot description, URDF)
Before this commit: robot iiwa14, 15 links, 14 joints
Links:
- removed link adaptor_kuka
- removed link end_effector
- added link adapter, mass 1; visual mesh filename=meshes/iiwa14/visual/schunk_adapter-Assembly_simplified.stl scale=0.001 0.001 0.001
- added link iiwa_link_ee, mass 0.000001
- link end_effector_sponge: geometry visual mesh filename=meshes/iiwa14/visual/adaptor_endeffector-Body_simplified.stl scale=0.001 0.001 0.001
- link force_torque_sensor: geometry visual mesh filename=meshes/iiwa14/visual/ATI-Delta_simplified.stl scale=0.001 0.001 0.001
Joints:
- removed joint force_torque_sensor_mount
- removed joint iiwa_joint_8
- added joint iiwa_joint_ee: type fixed, parent iiwa_link_7, child iiwa_link_ee, origin xyz=0 0 0.045 rpy=0 0 0
- added joint iiwa_joint_ft: type fixed, parent iiwa_link_ee, child force_torque_sensor, origin xyz=0 0 0 rpy=0 0 1.57
- joint end_effector_joint: child end_effector -> adapter; origin xyz=0 0 0.02 rpy=0 0 0.0 -> xyz=0 0 0.033 rpy=0 0 0.0
- joint end_effector_joint_sponge: origin xyz=0 0 0.015 rpy=0 0 0.0 -> xyz=0 0 0.078 rpy=0 0 0.0; parent end_effector -> adapter

Commit message: change the robot urdf file back to the real robot without end-effector offset

File: robots/kuka_iiwa/iiwa14.urdf (robot description, URDF)
Before this commit: robot iiwa14, 15 links, 14 joints
Joints:
- joint end_effector_joint_sponge: origin xyz=0 0 0.078 rpy=0 0 0.0 -> xyz=0 0 0.058 rpy=0 0 0.0

File: robots/kuka_iiwa/iiwa14_visual.urdf (robot description, URDF)
Before this commit: robot iiwa14, 15 links, 14 joints
Joints:
- joint end_effector_joint_sponge: origin xyz=0 0 0.078 rpy=0 0 0.0 -> xyz=0 0 0.058 rpy=0 0 0.0
