Commit message: Modify iiwa urdf and add srdf

File: ros_pybullet_interface_examples/robots/kuka_iiwa/iiwa14.urdf (robot description, URDF)
Before this commit: robot iiwa14, 13 links, 12 joints
Links:
- link adaptor_kuka: geometry collision mesh filename=package://ros_pybullet_interface_examples/robots/kuka_iiwa/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 scale=0.001 0.001 0.001; visual mesh filename=package://ros_pybullet_interface_examples/robots/kuka_iiwa/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 scale=0.001 0.001 0.001
- link end_effector: geometry collision mesh filename=package://ros_pybullet_interface_examples/robots/kuka_iiwa/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 scale=0.001 0.001 0.001; visual mesh filename=package://ros_pybullet_interface_examples/robots/kuka_iiwa/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 scale=0.001 0.001 0.001
- link force_torque_sensor: geometry collision cylinder length=0.0333 radius=0.04; visual mesh filename=package://ros_pybullet_interface_examples/robots/kuka_iiwa/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 scale=0.001 0.001 0.001
- link iiwa_link_0: geometry collision mesh filename=package://ros_pybullet_interface_examples/robots/kuka_iiwa/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; visual mesh filename=package://ros_pybullet_interface_examples/robots/kuka_iiwa/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
- link iiwa_link_1: geometry collision mesh filename=package://ros_pybullet_interface_examples/robots/kuka_iiwa/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; visual mesh filename=package://ros_pybullet_interface_examples/robots/kuka_iiwa/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
- link iiwa_link_2: geometry collision mesh filename=package://ros_pybullet_interface_examples/robots/kuka_iiwa/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; visual mesh filename=package://ros_pybullet_interface_examples/robots/kuka_iiwa/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
- link iiwa_link_3: geometry collision mesh filename=package://ros_pybullet_interface_examples/robots/kuka_iiwa/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; visual mesh filename=package://ros_pybullet_interface_examples/robots/kuka_iiwa/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
- link iiwa_link_4: geometry collision mesh filename=package://ros_pybullet_interface_examples/robots/kuka_iiwa/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; visual mesh filename=package://ros_pybullet_interface_examples/robots/kuka_iiwa/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
- link iiwa_link_5: geometry collision mesh filename=package://ros_pybullet_interface_examples/robots/kuka_iiwa/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; visual mesh filename=package://ros_pybullet_interface_examples/robots/kuka_iiwa/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
- link iiwa_link_6: geometry collision mesh filename=package://ros_pybullet_interface_examples/robots/kuka_iiwa/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; visual mesh filename=package://ros_pybullet_interface_examples/robots/kuka_iiwa/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
- link iiwa_link_7: geometry collision mesh filename=package://ros_pybullet_interface_examples/robots/kuka_iiwa/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; visual mesh filename=package://ros_pybullet_interface_examples/robots/kuka_iiwa/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
