Commit message: test with Kuka example

File: rpbi_examples/robots/kuka_lwr.urdf (robot description, URDF)
Before this commit: robot lwr, 9 links, 8 joints
Links:
- removed link lwr_arm_2_link
- removed link lwr_arm_3_link
- removed link lwr_arm_4_link
- removed link lwr_arm_5_link
- removed link lwr_arm_6_link
- removed link lwr_arm_7_link
- link base: geometry visual box size=1 1 0.04
- link lwr_arm_0_link: geometry visual box size=0.08 0.12 0.06; visual cylinder length=0.1 radius=0.06
- link lwr_arm_1_link: geometry visual cylinder length=0.05 radius=0.03; visual cylinder length=0.1 radius=0.06
Joints:
- removed joint lwr_arm_1_joint
- removed joint lwr_arm_2_joint
- removed joint lwr_arm_3_joint
- removed joint lwr_arm_4_joint
- removed joint lwr_arm_5_joint
- removed joint lwr_arm_6_joint
- joint lwr_arm_0_joint: axis 0 0 1 -> (none); limit lower=-2.96705972839 upper=2.96705972839 effort=204 velocity=1.91986217719 -> (none); type revolute -> fixed
